File: Hardware/gcvideo_lite_09/gcvideo_lite.kicad_pcb (KiCad board)
At the start: 4 copper layers, 49 x 30 mm, 44 parts, among them P1 CONN_11X2, P2 CONN_5, P3 CONN_4, P4 CONN_6, P5 CONN_2X2, P6 CONN_1, P7 CONN_1, P8 CONN_1, P9 CONN_1, U1 MachXO2-256-TQ100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

Commit message: update kicad files and replace cdk3404 with adv1725
Parts:
- removed C1, C17, C18, C2, C20, C21, C3, C4, C5: 100n, SMD_Packages:SM0805
- removed C10, C11, C12, C13, C14, C15, C16, C19, C7, C8, C9: 10n, SMD_Packages:SM0805
- removed C22, C6: 10u, SMD_Packages:SM1206POL
- removed JP1: RGB/COMP, SOLDER_JUMPER:SOLDER_JUMPER
- removed L1: INDUCTOR, SMD_Packages:SM0805
- removed P1: CONN_11X2, Pin_Headers:Pin_Header_Straight_2x11
- removed P2: CONN_5, Connect:SIL-5
- removed P3: CONN_4, Connect:SIL-4
- removed P4: CONN_6, Connect:SIL-6
- removed P5: CONN_2X2, Pin_Headers:Pin_Header_Straight_2x02
- removed P6, P7, P8, P9: CONN_1, Wire_Pads:SolderWirePad_single_0-8mmDrill
- removed R1: 348, SMD_Packages:SM0805
- removed R2, R3, R4, R5: 75, SMD_Packages:SM0805
- removed R6: 100, SMD_Packages:SM0805
- removed R7, R8: 4k7, SMD_Packages:SM0805
- removed U1: MachXO2-256-TQ100, SMD_Packages:TQFP_100
- removed U2: CDK3404, Housings_QFP:lqfp-48
- removed U4: 74LVC14, Housings_SOIC:SOIC-14_Narrow
Routing:
- net GND: track 116.1 -> 0.00 mm, vias 16 -> 0
- net +3.3V: track 82.8 -> 0.00 mm, vias 7 -> 0
- net /EXTCSYNCn: track 52.4 -> 0.00 mm, vias 1 -> 0
- net /EXTVSYNCn: track 48.8 -> 0.00 mm, vias 1 -> 0
- net /EXTHSYNCn: track 45.7 -> 0.00 mm, vias 1 -> 0
- net /DACCLOCK: track 31.5 -> 0.00 mm, vias 2 -> 0
- net /B7: track 31.1 -> 0.00 mm, vias 2 -> 0
- net /CLK54: track 28.8 -> 0.00 mm, vias 1 -> 0
- net /B6: track 28.4 -> 0.00 mm, vias 2 -> 0
- net /B5: track 26.1 -> 0.00 mm, vias 2 -> 0
- net /B4: track 23.7 -> 0.00 mm, vias 2 -> 0
- net +3.3VDAC: track 23.2 -> 0.00 mm, vias 4 -> 0
- net /B3: track 21.3 -> 0.00 mm, vias 2 -> 0
- net /VSYNC: track 21.3 -> 0.00 mm
- net /HSYNC: track 20.7 -> 0.00 mm
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- removed copper zone on Inner1.Cu, net +3.3V
- removed copper zone on Inner1.Cu, net +3.3VDAC
- removed copper zone on Inner2.Cu, net GND
Other:
- board outline removed
- net class Default: clearance 0.1778 -> 0.1524; trace_width 0.2032 -> 0.1524; via_dia 1.27 -> 0.508; via_drill 0.635 -> 0.254
- net class Power removed
- rule pad_to_mask_clearance: 0 -> 0.0508
- rule trace_clearance: 0.1778 -> 0.1524
- rule trace_min: 0.2032 -> 0.1524
- rule via_min_drill: 0.508 -> 0.254
- rule via_min_size: 0.889 -> 0.508
- board text removed: "-ik"
- board text removed: "B"
- board text removed: "B-G-R"
- board text removed: "C V H -"
- board text removed: "CS"
- board text removed: "G"
- board text removed: "GCVideo Lite 0.9"
- board text removed: "GND"
- board text removed: "HS"
- board text removed: "JTAG"
- board text removed: "R"
- board text removed: "RGB"
- board text removed: "SPARE"
- board text removed: "VS"
